File: ISPnub-Stick.kicad_pcb (KiCad board)
At the start: 2 copper layers, 74 x 26 mm, 13 parts, among them SW1 SW_Push, SW2 SW_SPDT, U1 ATmega1284P-A, X1 Conn_02x03_Counter_Clockwise

Commit message: rev1.0 changes
Parts:
- added REF**: KiCad-Logo2_5mm_Copper, Symbol:KiCad-Logo2_5mm_Copper, B.Cu at (72.6, 94.0)
- added REF**: OSHW-Logo_5.7x6mm_Copper, Symbol:OSHW-Logo_5.7x6mm_Copper, B.Cu at (72.6, 101.5)
- SW1: footprint Button_Switch_SMD:SW_SPST_Omron_B3FS-100xP -> ALITECS:TS-1187A-B-A-B
- moved D2 0.11 mm to (71.1, 105.9)
- moved R3 0.10 mm to (74.3, 105.9)
Routing:
- net Net-(U1-PD3): track 11.6 -> 10.9 mm
Other:
- outline, holes or cut-outs redrawn
- board text added: "${TITLE} REV ${REVISION}"
- board text added: "https://github.com/Alex9779/ISPnub-Stick.git"
- board text removed: "${TITLE} v${REVISION}"
