File: ISPnub-Stick.kicad_sch (KiCad schematic)
At the start: 13 parts, among them SW1 SW_Push, SW2 SW_SPDT, U1 ATmega1284P-A, X1 Conn_02x03_Counter_Clockwise

Commit message: rev1.0 changes
Parts:
- SW1: footprint Button_Switch_SMD:SW_SPST_Omron_B3FS-100xP -> ALITECS:TS-1187A-B-A-B; JLCPCB Part # C87038 -> C318884
- X1: now not fitted; now left out of the parts list
Changed lines of the file:
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@@
   )
   (symbol (lib_id "Connector_Generic:Conn_02x03_Odd_Even") (at 180.34 34.29 0) (unit 1)
-    (in_bom yes) (on_board yes) (dnp no) (fields_autoplaced)
+    (in_bom no) (on_board yes) (dnp yes) (fields_autoplaced)
     (property "Reference" "X1" (at 181.61 25.4 0)
       (effects (font (size 1.27 1.27)))
@@
       (effects (font (size 1.27 1.27)))
     )
-    (property "Footprint" "Button_Switch_SMD:SW_SPST_Omron_B3FS-100xP" (at 110.49 133.35 0)
+    (property "Footprint" "ALITECS:TS-1187A-B-A-B" (at 110.49 133.35 0)
       (effects (font (size 1.27 1.27)) hide)
     )
@@
       (effects (font (size 1.27 1.27)) hide)
     )
-    (property "JLCPCB Part #" "C87038" (at 110.49 138.43 0)
-      (effects (font (size 1.27 1.27)) hide)
-    )
+    (property "JLCPCB Part #" "C318884" (at 110.49 138.43 0)
+      (effects (font (size 1.27 1.27)) hide)
+    )
